Commit message: modify

File: vistar_gazebo/models/cube_marker/cube_marker.urdf (robot description, URDF)
Before this commit: robot cube_marker, 1 links, 0 joints
Links:
- removed link cube_marker
- added link cube_marker_link, mass 0.25; collision box size=0.06 0.06 0.06; visual mesh filename=package://vistar_gazebo/models/cube_marker/meshes/artag.dae

File: vistar_gazebo/models/kinect/kinect.xacro (robot description, xacro)
@@ -30,11 +30,10 @@
             </collision>
         </link>
-<!--
-<joint name="camera_depth_joint" type="fixed">
+<!--<joint name="${prefix}_depth_joint" type="fixed">
     <origin xyz="0 0.011 0" rpy="0 0 0" />
-    <parent link="camera_link" />
-    <child link="camera_depth_frame" />
+    <parent link="${prefix}_link" />
+    <child link="${prefix}_depth_frame" />
   </joint>
-  <link name="camera_depth_frame">
+  <link name="${prefix}_depth_frame">
     <inertial>
       <mass value="0.01" />
@@ -45,10 +44,10 @@
     </inertial>
   </link>
-  <joint name="camera_depth_optical_joint" type="fixed">
-    <origin xyz="0 0 0" rpy="${-M_PI/2} 0 ${-M_PI/2}" />
-    <parent link="camera_depth_frame" />
-    <child link="camera_depth_optical_frame" />
+  <joint name="${prefix}_depth_optical_joint" type="fixed">
+    <origin xyz="0 0 0" rpy="${-pi/2} 0 ${-pi/2}" />
+    <parent link="${prefix}_depth_frame" />
+    <child link="${prefix}_depth_optical_frame" />
   </joint>
-  <link name="camera_depth_optical_frame">
+  <link name="${prefix}_depth_optical_frame">
     <inertial>
       <mass value="0.001" />
@@ -59,10 +58,10 @@
     </inertial>
   </link>
-  <joint name="camera_rgb_joint" type="fixed">
+  <joint name="${prefix}_rgb_joint" type="fixed">
     <origin xyz="0 -0.012 0" rpy="0 0 0" />
-    <parent link="camera_link" />
-    <child link="camera_rgb_frame" />
+    <parent link="${prefix}_link" />
+    <child link="${prefix}_rgb_frame" />
   </joint>
-  <link name="camera_rgb_frame">
+  <link name="${prefix}_rgb_frame">
     <inertial>
       <mass value="0.001" />
@@ -73,10 +72,10 @@
     </inertial>
   </link>
-  <joint name="camera_rgb_optical_joint" type="fixed">
-    <origin xyz="0 0 0" rpy="${-M_PI/2} 0 ${-M_PI/2}" />
-    <parent link="camera_rgb_frame" />
-    <child link="camera_rgb_optical_frame" />
+  <joint name="${prefix}_rgb_optical_joint" type="fixed">
+    <origin xyz="0 0 0" rpy="${-pi/2} 0 ${-pi/2}" />
+    <parent link="${prefix}_rgb_frame" />
+    <child link="${prefix}_rgb_optical_frame" />
   </joint>
-  <link name="camera_rgb_optical_frame">
+  <link name="${prefix}_rgb_optical_frame">
     <inertial>
       <mass value="0.001" />
@@ -87,5 +86,5 @@
     </inertial>
   </link>
-  -->
+-->
         <gazebo reference="${prefix}_link">
             <sensor type="depth" name="${prefix}">
