Commit message: modify

File: vistar_description/urdf/vistar_with_camera.xacro (robot description, xacro)
@@ -8,5 +8,5 @@
 		<parent link="world" />
 		<child link = "base_link" />
-		<origin xyz="0.0 0.0 1.015" rpy="0.0 0.0 0.0" />
+		<origin xyz="0.375 0.0 1.015" rpy="0.0 0.0 0.0" />
 	</joint>
 	<xacro:ur3_robot prefix="" joint_limited="false"/>
