Commit message: 删掉碍事的table，使用box来代替，c++规划成功

File: vistar_description/urdf/vistar_with_topkinect.xacro (robot description, xacro)
@@ -8,11 +8,11 @@
 		<parent link="world" />
 		<child link = "base_link" />
-		<origin xyz="0 0 1.05" rpy="0.0 0.0 0.0" />
+		<origin xyz="0 0 0.45" rpy="0.0 0.0 0.0" />
 	</joint>
 	<xacro:ur3_robot prefix="" joint_limited="false"/>
 	<!-- Robotiq from Beta Robots fork-->
 	<xacro:include filename="$(find robotiq_2f_85_gripper_description)/urdf/robotiq_2f_85.urdf.xacro" />
-	<xacro:robotiq_2f_85 name="gripper" parent="ee_link" precise_collision="false" adaptive_transmission="false">
-		<origin xyz="0 0 0" rpy="${pi/2} ${pi/2} ${pi/2}" />
+	<xacro:robotiq_2f_85 name="gripper" parent="tool0" precise_collision="true" adaptive_transmission="false">
+		<origin xyz="0 0 0" rpy="0 0 ${pi/2}" />
 	</xacro:robotiq_2f_85>
 	<!-- kinect -->

File: vistar_gazebo/urdf/vistar_with_topkinect.urdf (robot description, URDF)
Before this commit: robot vistar, 24 links, 23 joints
Links:
- link gripper_base: geometry collision mesh filename=package://robotiq_2f_85_gripper_description/meshes/collisio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 scale=0.001 0.001 0.001; visual mesh filename=package://robotiq_2f_85_gripper_description/meshes/visual/b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
- link gripper_left_coupler: geometry collision mesh filename=package://robotiq_2f_85_gripper_description/meshes/collisio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 scale=0.001 0.001 0.001; visual mesh filename=package://robotiq_2f_85_gripper_description/meshes/visual/c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 scale=0.001 0.001 0.001
- link gripper_left_driver: geometry collision mesh filename=package://robotiq_2f_85_gripper_description/meshes/collisio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 scale=0.001 0.001 0.001; visual mesh filename=package://robotiq_2f_85_gripper_description/meshes/visual/d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 scale=0.001 0.001 0.001
- link gripper_left_follower: geometry collision mesh filename=package://robotiq_2f_85_gripper_description/meshes/collisio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 scale=0.001 0.001 0.001; visual mesh filename=package://robotiq_2f_85_gripper_description/meshes/visual/f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 scale=0.001 0.001 0.001
- link gripper_left_pad: geometry collision mesh filename=package://robotiq_2f_85_gripper_description/meshes/collisio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 scale=0.001 0.001 0.001; visual mesh filename=package://robotiq_2f_85_gripper_description/meshes/visual/p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 scale=0.001 0.001 0.001
- link gripper_left_spring_link: geometry collision mesh filename=package://robotiq_2f_85_gripper_description/meshes/collisio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 scale=0.001 0.001 0.001; visual mesh filename=package://robotiq_2f_85_gripper_description/meshes/visual/s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 scale=0.001 0.001 0.001
- link gripper_right_coupler: geometry collision mesh filename=package://robotiq_2f_85_gripper_description/meshes/collisio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 scale=0.001 0.001 0.001; visual mesh filename=package://robotiq_2f_85_gripper_description/meshes/visual/c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 scale=0.001 0.001 0.001
- link gripper_right_driver: geometry collision mesh filename=package://robotiq_2f_85_gripper_description/meshes/collisio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 scale=0.001 0.001 0.001; visual mesh filename=package://robotiq_2f_85_gripper_description/meshes/visual/d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 scale=0.001 0.001 0.001
- link gripper_right_follower: geometry collision mesh filename=package://robotiq_2f_85_gripper_description/meshes/collisio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 scale=0.001 0.001 0.001; visual mesh filename=package://robotiq_2f_85_gripper_description/meshes/visual/f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 scale=0.001 0.001 0.001
- link gripper_right_pad: geometry collision mesh filename=package://robotiq_2f_85_gripper_description/meshes/collisio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 scale=0.001 0.001 0.001; visual mesh filename=package://robotiq_2f_85_gripper_description/meshes/visual/p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 scale=0.001 0.001 0.001
- link gripper_right_spring_link: geometry collision mesh filename=package://robotiq_2f_85_gripper_description/meshes/collisio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 scale=0.001 0.001 0.001; visual mesh filename=package://robotiq_2f_85_gripper_description/meshes/visual/s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 scale=0.001 0.001 0.001
Joints:
- removed joint ee_link_gripper_base_joint
- added joint tool0_gripper_base_joint: type fixed, parent tool0, child gripper_base, origin xyz=0 0 0 rpy=0 0 1.57079632679
