Commit message: 仿真环境和识别的最后修改

File: robotiq_2f_85_gripper_description/urdf/robotiq_2f_85.urdf.xacro (robot description, xacro)
@@ -442,30 +442,44 @@
 				</actuator>
 			</transmission>
-			<gazebo>
-				<plugin name="${name}_right_follower_joint_plugin" filename="libroboticsgroup_gazebo_mimic_joint_plugin.so">
-					<joint>${name}_right_driver_joint</joint>
-					<mimicJoint>${name}_right_follower_joint</mimicJoint>
-					<multiplier>-1</multiplier>
-				</plugin>
-				<plugin name="${name}_right_spring_link_joint_plugin" filename="libroboticsgroup_gazebo_mimic_joint_plugin.so">
-					<joint>${name}_right_driver_joint</joint>
-					<mimicJoint>${name}_right_spring_link_joint</mimicJoint>
-					<multiplier>1</multiplier>
-				</plugin>
-				<plugin name="${name}_left_follower_joint_plugin" filename="libroboticsgroup_gazebo_mimic_joint_plugin.so">
-					<joint>${name}_right_driver_joint</joint>
-					<mimicJoint>${name}_left_follower_joint</mimicJoint>
-					<multiplier>-1</multiplier>
-				</plugin>
-				<plugin name="${name}_left_spring_link_joint_plugin" filename="libroboticsgroup_gazebo_mimic_joint_plugin.so">
-					<joint>${name}_right_driver_joint</joint>
-					<mimicJoint>${name}_left_spring_link_joint</mimicJoint>
-					<multiplier>1</multiplier>
-				</plugin>
-				<plugin name="${name}_left_driver_joint_plugin" filename="libroboticsgroup_gazebo_mimic_joint_plugin.so">
-					<joint>${name}_right_driver_joint</joint>
-					<mimicJoint>${name}_left_driver_joint</mimicJoint>
-					<multiplier>1</multiplier>
-				</plugin>
+		<gazebo>
+			<plugin name="${name}_right_follower_joint_plugin" filename="libroboticsgroup_gazebo_mimic_joint_plugin.so">
+				<joint>${name}_right_driver_joint</joint>
+				<mimicJoint>${name}_right_follower_joint</mimicJoint>
+				<multiplier>-1</multiplier>
+			</plugin>
+			<plugin name="${name}_right_spring_link_joint_plugin" filename="libroboticsgroup_gazebo_mimic_joint_plugin.so">
+				<joint>${name}_right_driver_joint</joint>
+				<mimicJoint>${name}_right_spring_link_joint</mimicJoint>
+				<multiplier>1</multiplier>
+			</plugin>
+			<plugin name="${name}_left_follower_joint_plugin" filename="libroboticsgroup_gazebo_mimic_joint_plugin.so">
+				<joint>${name}_right_driver_joint</joint>
+				<mimicJoint>${name}_left_follower_joint</mimicJoint>
+				<multiplier>-1</multiplier>
+			</plugin>
+			<plugin name="${name}_left_spring_link_joint_plugin" filename="libroboticsgroup_gazebo_mimic_joint_plugin.so">
+				<joint>${name}_right_driver_joint</joint>
+				<mimicJoint>${name}_left_spring_link_joint</mimicJoint>
+				<multiplier>1</multiplier>
+			</plugin>
+			<plugin name="${name}_left_driver_joint_plugin" filename="libroboticsgroup_gazebo_mimic_joint_plugin.so">
+				<joint>${name}_right_driver_joint</joint>
+				<mimicJoint>${name}_left_driver_joint</mimicJoint>
+				<multiplier>1</multiplier>
+			</plugin>
+		</gazebo>
+		<gazebo reference="${name}_right_pad">
+		    <implicitSpringDamper>1</implicitSpringDamper>
+		    <mu1>100000</mu1>
+		    <mu2>100000</mu2>
+		    <kp>100000000.0</kp>
+		    <kd>1.0</kd>
+		</gazebo>
+		<gazebo reference="${name}_left_pad">
+		    <implicitSpringDamper>1</implicitSpringDamper>
+		    <mu1>100000</mu1>
+		    <mu2>100000</mu2>
+		    <kp>100000000.0</kp>
+		    <kd>1.0</kd>
 		</gazebo>
 	</xacro:unless>

File: vistar_description/urdf/vistar_with_kinect.xacro (robot description, xacro)
@@ -8,5 +8,5 @@
 		<parent link="world" />
 		<child link = "base_link" />
-		<origin xyz="0.0 0.0 0.0" rpy="0.0 0.0 0.0" />
+		<origin xyz="0 0 1.015" rpy="0.0 0.0 0.0" />
 	</joint>
 	<xacro:ur3_robot prefix="" joint_limited="false"/>
@@ -18,6 +18,32 @@
 	<!-- kinect -->
 	<xacro:include filename="$(find vistar_gazebo)/models/kinect/kinect.xacro"/>
-	<xacro:kinect_camera prefix="camera" parent="world" >
-		<origin xyz="0.8 0.7 0.03" rpy="0 0 ${pi}" />
+	<joint name="world_root_fixed" type="fixed">
+		<origin xyz="0 1.1 0.51" rpy="0 0 0"/>
+		<parent link="world"/>
+		<child link="root_link"/>
+	</joint>
+	<link name="root_link">
+	<visual>
+		<origin xyz="0 0 0" rpy="0 0 0"/>
+		<geometry>
+			<box size="0.1 0.1 1.02"/>
+		</geometry>
+	</visual>
+	<collision>
+		<origin xyz="0 0 0" rpy="0 0 0"/>
+		<geometry>
+			<box size="0.1 0.1 1.02"/>
+		</geometry>
+	</collision>
+	<inertial>
+		<mass value="1e2" />
+		<origin xyz="0.0 0.0 0.0" />
+		<inertia ixx = "0.000001" ixy = "0.000000" ixz = "0.000000"
+				iyx = "0.000000" iyy = "0.000001" iyz = "0.000000"
+				izx = "0.000000" izy = "0.000000" izz = "0.000001" />
+	</inertial>
+	</link>
+	<xacro:kinect_camera prefix="camera" parent="root_link" >
+		<origin xyz="0 0 0.535" rpy="0 0 ${-pi/2}" />
 	</xacro:kinect_camera>
        <!-- Plugin -->

File: vistar_gazebo/models/kinect/kinect.xacro (robot description, xacro)
@@ -17,11 +17,4 @@
                 </geometry>
             </visual>
-            <inertial>
-                <mass value="0.01" />
-                <origin xyz="0 0 0" />
-                <inertia ixx="0.001" ixy="0.0" ixz="0.0"
-                        iyy="0.001" iyz="0.0"
-                        izz="0.001" />
-            </inertial>
             <collision>
                 <geometry>
@@ -30,61 +23,10 @@
             </collision>
         </link>
-<!--<joint name="${prefix}_depth_joint" type="fixed">
-    <origin xyz="0 0.011 0" rpy="0 0 0" />
-    <parent link="${prefix}_link" />
-    <child link="${prefix}_depth_frame" />
-  </joint>
-  <link name="${prefix}_depth_frame">
-    <inertial>
-      <mass value="0.01" />
-      <origin xyz="0 0 0" />
-      <inertia ixx="0.001" ixy="0.0" ixz="0.0"
-        iyy="0.001" iyz="0.0"
-        izz="0.001" />
-    </inertial>
-  </link>
-  <joint name="${prefix}_depth_optical_joint" type="fixed">
-    <origin xyz="0 0 0" rpy="${-pi/2} 0 ${-pi/2}" />
-    <parent link="${prefix}_depth_frame" />
-    <child link="${prefix}_depth_optical_frame" />
-  </joint>
-  <link name="${prefix}_depth_optical_frame">
-    <inertial>
-      <mass value="0.001" />
-      <origin xyz="0 0 0" />
-      <inertia ixx="0.0001" ixy="0.0" ixz="0.0"
-        iyy="0.0001" iyz="0.0"
-        izz="0.0001" />
-    </inertial>
-  </link>
-  <joint name="${prefix}_rgb_joint" type="fixed">
-    <origin xyz="0 -0.012 0" rpy="0 0 0" />
-    <parent link="${prefix}_link" />
-    <child link="${prefix}_rgb_frame" />
-  </joint>
-  <link name="${prefix}_rgb_frame">
-    <inertial>
-      <mass value="0.001" />
-      <origin xyz="0 0 0" />
-      <inertia ixx="0.0001" ixy="0.0" ixz="0.0"
-        iyy="0.0001" iyz="0.0"
-        izz="0.0001" />
-    </inertial>
-  </link>
-  <joint name="${prefix}_rgb_optical_joint" type="fixed">
-    <origin xyz="0 0 0" rpy="${-pi/2} 0 ${-pi/2}" />
-    <parent link="${prefix}_rgb_frame" />
-    <child link="${prefix}_rgb_optical_frame" />
-  </joint>
-  <link name="${prefix}_rgb_optical_frame">
-    <inertial>
-      <mass value="0.001" />
-      <origin xyz="0 0 0" />
-      <inertia ixx="0.0001" ixy="0.0" ixz="0.0"
-        iyy="0.0001" iyz="0.0"
-        izz="0.0001" />
-    </inertial>
-  </link>
--->
+        <joint name="${prefix}_optical_joint" type="fixed">
+            <origin xyz="0 0 0" rpy="-1.5708 0 -1.5708"/>
+            <parent link="${prefix}_link"/>
+            <child link="${prefix}_frame_optical"/>
+        </joint>
+        <link name="${prefix}_frame_optical"/>
         <gazebo reference="${prefix}_link">
             <sensor type="depth" name="${prefix}">
@@ -112,5 +54,5 @@
                     <cameraInfoTopicName>rgb/camera_info</cameraInfoTopicName>
                     <depthImageCameraInfoTopicName>depth/camera_info</depthImageCameraInfoTopicName>
-                    <frameName>${prefix}_link</frameName>
+                    <frameName>${prefix}_frame_optical</frameName>
                     <baseline>0.1</baseline>
                     <distortion_k1>0.0</distortion_k1>
